File: Eagle/Display Shield/Small e-PaperShield v2.1.brd (EAGLE design)
At the start: 106.3 x 56.3 mm, 118 parts, among them J2 3300060P1-ST-TF-003A, J3 2.54-8p-male-SMD, J4 2.54-8p-male-SMD, J5 2.54-6p-male-SMD, J6 2.54-6p-male-SMD, J7 2.54-2x3p-female-SMD, Q10 MOSFET-P-044021001, Q11 2N7002, Q2 2N7002, Q3 MOSFET-P-044021001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

Commit message: finished display shield
Parts:
- removed J4: 2.54-8p-male-SMD, Connector:8P-2.54-SMD
- added U$1: SMD-BLUE-MALE-HEADER-R/A(3P-2.54), Seeed-OPL-Connector:H3-SMD-2.54
- moved JP1 78.7 mm to (88.4, 58.2)
- moved R15 78.7 mm to (93.4, 52.4)
- moved R5 78.7 mm to (86.2, 52.4)
- moved R17 78.7 mm to (97.0, 52.4)
- moved R6 78.7 mm to (89.8, 52.4)
Connections:
- net GND: no longer J4.7
- net M_/EPD_CS: now also U$1.3; no longer J4.3
- net M_/WORD_STOCK_CS: now also U$1.2; no longer J4.2
- net M_EPD_DISCHARGE: now also U$1.1; no longer J4.1
Routing:
- net BTN2: track 98.5 -> 166.8 mm
- net BTN0: track 108.0 -> 170.8 mm, vias 1 -> 4
- net BTN1: track 185.9 -> 129.9 mm, vias 2 -> 3
- net BTN3: track 172.9 -> 139.1 mm, vias 3 -> 1
- net M_VCC_3V3: track 77.5 -> 92.7 mm, vias 2 -> 0

Commit message: final gerber files for display shield
Parts:
- moved S6 6.40 mm to (7.05, 26.0)
- moved S5 3.61 mm to (94.5, 26.1)
- moved S7 3.16 mm to (96.5, 40.8)
- moved S8 2.00 mm to (5.05, 40.8)
- moved JP1 1.57 mm to (86.8, 58.3)
Routing:
- net BTN3: track 139.1 -> 169.0 mm
- net BTN1: track 129.9 -> 159.0 mm, vias 3 -> 0
- net BTN0: track 170.8 -> 192.8 mm, vias 4 -> 1
- net BTN2: track 166.8 -> 147.6 mm, vias 4 -> 1
- net VCC_3V3_EPD: track 57.2 -> 72.6 mm, vias 4 -> 6
- net LED0: track 11.0 -> 7.42 mm
Other:
- board size 106.3 x 56.3 mm -> 100.3 x 56.2 mm
- board text removed: "/Users/raffael/Desktop/EPFL Master/CHIC/dOry_logo_mono.bmp"
- board text removed: "D13"
